File: CIMs/Lipmouse_CIM/PCB-design/Lipmouse_Teensy/Lipmouse_Teensy.sch (EAGLE design)
At the start: 40 parts, among them IC1 AT90USB1286-MU, Q1 FDN360P, SW1 SPST_TACT-EVQQ2, SW2 SPST_TACT-EVQQ2, U2 MCP73831, X1 MINI-USB-32005-201

Commit message: Update Lipsy (Lipmouse) PCB and case designs
Parts:
- removed C10, C8: 4.7u, resistor:C-EUC0805
- removed C12, C14, C5: 1u, resistor:C-EUC0603
- removed C13, C15, C3, C4: 100n, resistor:C-EUC0603
- removed C6, C7: 18p, resistor:C-EUC0603
- removed CRYSTAL: 16MHz, SparkFun-FreqCtrl:CRYSTALTXC-7A
- removed D1: (no value), eagle-ltspice:SCHOTTKY-DIODE
- removed IC1: AT90USB1286-MU, Sensorboard:AT90USB1287-AU
- removed JP2: M02-JST-2MM-SMT, SparkFun-Connectors:M02-JST-2MM-SMT
- removed JP3: NC, pinhead:PINHD-2X5
- removed L1, L2: (no value), WE-CBF:WE-CBF-74279201_0805
- removed MCP1703: MCP1703-3302E/DB, Microchip_By_element14_Batch_1:MCP1703-3302E/DB
- removed MP3V7007: MP3V7007GP, my_own_designs:MP3V7007GP
- removed Q1: FDN360P, transistor-power:FDN360P
- removed R11: 330, resistor:R-EU_R0603
- removed SJ1: (no value), jumper:SJ
- removed SW1, SW2: SPST_TACT-EVQQ2, adafruit:SPST_TACT-EVQQ2
- removed U$1: BLE-HM-10, Random parts:BLE-HM-10
- removed U2: MCP73831, SparkFun:MCP73831
- removed X1: MINI-USB-32005-201, con-cypressindustries:MINI-USB-32005-201
- added C2: 100nF, resistor:C-EUC0805K
- added LED5, LED6, LED7: TSAL6200, led:LED5MM
- added PAD6, PAD7: (no value), wirepad:1,6/0,9
- added R5, R6: 470R, resistor:R-EU_R0805W
- added S1, S2: (no value), adafruit:31-XX
- added SV1: (no value), con-lsta:FE05-1
- added SV2: (no value), con-harting-ml:ML6
- added TEENSY++: C-TEENSY-LIPMOUSE, teensy_lipmouse:C-TEENSY-LIPMOUSE
- added U$2: MP3V7007GP, libMP3V7007GP:MP3V7007GP
- added U$3: TSOP4838, TSOPXXXX:TSOP48XX
- C1: value 10n -> 100nF; device resistor:C-EUC0603 -> resistor:C-EUC0805K
- LED1, LED2, LED3: device led:LEDSMT1206 -> adafruit:LED3MM
- R1: value 330 -> 10k; device resistor:R-EU_R0603 -> resistor:R-EU_R0805W
- R10: value 470 -> 180R; device resistor:R-EU_R0603 -> resistor:R-EU_R0805W
- R2, R3: value 4k7 -> 10k; device resistor:R-EU_R0603 -> resistor:R-EU_R0805W
- R4: value 100k -> 10k; device resistor:R-EU_R0603 -> resistor:R-EU_R0805W
- R7: value 22 -> 470R; device resistor:R-EU_R0603 -> resistor:R-EU_R0805W
- R8: value 22 -> 180R; device resistor:R-EU_R0603 -> resistor:R-EU_R0805W
- R9: value 330 -> 180R; device resistor:R-EU_R0603 -> resistor:R-EU_R0805W
Connections:
- removed net +3V3: C14.1, C15.2, C3.1, IC1.VCC@1, IC1.VCC@2, JP3.4, L2.1, MCP1703.VOUT, MP3V7007.VCC, R2.1, U$1.3.3V
- removed net AVCC: C13.1, IC1.AVCC, L2.2
- removed net D+: R7.1, X1.3
- removed net D-: R8.1, X1.2
- removed net N$4: C5.2, IC1.UCAP
- removed net PF0: IC1.PF0(ADC0), MP3V7007.VOUT
- removed net PIO: R10.1, U$1.PIO1
- removed net PIO1: LED3.A, R10.2
- removed net RESETBT: IC1.PD7(T0), U$1.RESETB
- removed net RST: C1.1, IC1.RESET, JP3.6, R1.1, R2.2
- removed net RX: IC1.PD2(RXD1/INT2), U$1.UART_TX
- removed net SW1: R1.2, SW1.S
- removed net TCK: IC1.PF4(ADC4/TCK), JP3.1
- removed net TDI: IC1.PF7(ADC7/TDI), JP3.9
- removed net TDO: IC1.PF6(ADC6/TDO), JP3.3
- removed net TMS: IC1.PF5(ADC5/TMS), JP3.5
- removed net TX: IC1.PD3(TXD1/INT3), U$1.UART_RX
- removed net V+: C8.2, D1.C, IC1.UVCC, IC1.VBUS, L1.2, Q1.G, R11.1, R4.1, R9.2, U2.VIN
- removed net VBAT: C10.1, JP2.1, Q1.D, U2.VBAT
- removed net VSYS: C12.2, MCP1703.VIN, SJ1.2
- removed net XTAL1: C6.2, CRYSTAL.1, IC1.XTAL2
- removed net XTAL2: C7.2, CRYSTAL.2, IC1.XTAL1
- new net FSR1: R1.1, SV1.1, TEENSY++.ADC4,PF4
- new net FSR2: R2.1, SV1.4, TEENSY++.ADC5,PF5
- new net FSR3: R3.1, SV1.2, TEENSY++.ADC6,PF6
- new net FSR4: R4.1, SV1.5, TEENSY++.ADC7,PF7
- new net IR1: LED7.C, TEENSY++.XCK1,PD5
- new net IR2: LED6.C, TEENSY++.LED,T1,PD6
- new net IR3: LED5.C, TEENSY++.T0,PD7
- new net N$12: LED5.A, R10.2
- new net N$14: U$2.NC_2, U$2.NC_3, U$2.NC_4, U$2.NC_5
- new net N$8: LED2.C, TEENSY++.AIN1,INT7,PE7
- new net PB1: SV2.2, TEENSY++.RXD1,INT2,PD2
- new net PB2: SV2.5, TEENSY++.TXD1,INT3,PD3
- new net PB7: TEENSY++.OC1C,OC0A,PB7
- new net TSOP: TEENSY++.ICP1,PD4, U$3.OUT
- new net VCC: C1.1, C2.1, PAD6.P, R10.1, R5.2, R6.2, R7.2, R8.1, R9.1, SV1.3, SV2.3, SV2.6, TEENSY++.VCC, U$2.VCC, U$3.VCC
- net GND: now also C2.2, PAD7.P, R1.2, R2.2, S1.P, S2.P, SV2.1, SV2.4, TEENSY++.GND, TEENSY++.GND@1, TEENSY++.GND@2, U$2.GND, U$3.GND; no longer C10.2, C12.1, C13.2, C14.2, C15.1, C3.2, C4.1, C5.1, C6.1, C7.1, C8.1, IC1.GND@1, IC1.GND@2, IC1.GND@3, IC1.PE2(ALE/HWB), IC1.UGND, JP2.2, JP3.10, JP3.2, LED1.C, LED3.C, MCP1703.GND_(TAB), MCP1703.GND_(TAB)_2, MP3V7007.GND, SW1.P, SW1.P1, SW2.S, SW2.S1, U$1.GND1, U$1.GND2, U$1.GND3, U$1.GND4, U2.VSS, X1.5
- net N$1: now also LED1.A, R5.1; no longer L1.1, X1.1
- net N$10: now also LED7.A; no longer IC1.D-
- net N$11: now also LED6.A, R9.2; no longer LED1.A, R11.2
- net N$17: now also S1.S, TEENSY++._RST; no longer LED2.A, R9.1
- net N$2: now also LED2.A, R6.1; no longer LED2.C, U2.STAT
- net N$3: now also LED3.A, R7.1; no longer C4.2, IC1.AREF
- net N$5: now also S2.S, TEENSY++.T3,PC3; no longer IC1.PB0(SS/PCINT0), SW2.P, SW2.P1
- net N$6: now also LED1.C, TEENSY++.AIN0,INT6,PE6; no longer R3.1, U2.PROG
- net N$7: now also TEENSY++.ADC0,PF0, U$2.VOUT; no longer D1.A, Q1.S, SJ1.1
- net N$9: now also LED3.C, TEENSY++.SS,PB0; no longer IC1.D+, R7.2
Other:
- note removed: "3V3 LDO regulator"
- note removed: "HM-10 BLE module"
- note removed: "LiPo battery connector"
- note removed: "LiPo charger"
- note removed: "Lipmouse wireless PCB version 0.4"
- note removed: "MP3V7007GP Pressure Sensor"
- note removed: "Note: JTAG connector is also used for connection of the sensor signals to ADC pins connector must be mounted centered (because of short flatband cable leading to daugherboard) !"
- note removed: "charge current: 1000 / 4k7 = 212mA"
- note removed: "falllback jumper for power switch (in case too much sleep current)"
- note removed: "keep BT-module in reset during standby (sleep) ??"
- note removed: "open questions: *) sleep current (eg. leakage through sensors -> switch 3V3 via mosfet ?) *) find part: 90-deg leds (L1,L2,L3) *) find part: 90-deg pushbutton SW2 (+actuator) *) find part: JP2 (check with battery connector) *) smaller shottky diode or FETKEY for D1/Q1? *) pulldown for RESETBT ? *) check orientation of sensor/JTAG connector (matches daughterboard ?) *) check package/height and val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"
- note removed: "see microchip AN1149: battery charger and load sharing"
- note removed: "wakeup/usr/standby"
- moved on the sheet: C1, LED1, LED2, LED3, R1, R10, R2, R3, R4, R7, R8, R9
